File: pic_k42.brd (EAGLE design)
At the start: 152.6 x 75 mm, 70 parts, among them IC1 PIC18F57K42-E_PT, IC2 REF3440IDBVR, IC3 MAX232, IC4 ILAMP, K1 G6K-2P, Q1 ASF1, X1 RX-2, X10 J1, X11 22-23-2021, X2 TX-2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

Commit message: up
Parts:
- added LED1: +5, led:CHIPLED_1206
- added LED2: +15, led:CHIPLED_1206
- added LED4: -15, led:CHIPLED_1206
- added R13, R9: 3K, rcl:R1206
- added R8: 1K, rcl:R1206
- moved F1 9.79 mm to (82.6, 21.7)
Connections:
- removed net N$73: TP4.TP, X10.4
- removed net N$74: TP5.TP, X10.6
- new net N$75: LED1.A, R8.1
- new net N$78: LED2.A, R9.1
- new net N$82: LED4.C, R13.1
- new net N15: R13.2, TP5.TP, X10.6
- new net P15: R9.2, TP4.TP, X10.4
- net RAW_VDD: now also R8.2
- net VSS: now also LED1.C, LED2.C, LED4.A
Routing:
- net P15: track 0.00 -> 48.8 mm
- net N15: track 0.00 -> 47.3 mm
- net N$17: track 56.0 -> 90.3 mm, vias 1 -> 0
- net N$74: track 32.8 -> 0.00 mm
- net VDD: track 373.6 -> 405.1 mm, vias 6 -> 4
- net N$49: track 118.7 -> 147.9 mm
- net N$82: track 0.00 -> 29.2 mm
- net N$56: track 81.7 -> 55.1 mm
- net N$63: track 40.5 -> 65.8 mm
- net N$8: track 111.2 -> 86.2 mm
- net N$20: track 70.0 -> 93.0 mm
- net N$40: track 100.1 -> 119.8 mm, vias 1 -> 3
- net N$73: track 19.5 -> 0.00 mm
- net N$3: track 41.6 -> 60.3 mm, vias 2 -> 0
- net RAW_VDD: track 90.4 -> 107.5 mm, vias 0 -> 1
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