File: pic_k42.brd (EAGLE design)
At the start: 130.5 x 111.1 mm, 63 parts, among them IC1 PIC18F57K42-E_PT, IC2 REF3440IDBVR, IC3 MAX232, IC4 ILAMP, K1 G6K-2P, Q1 ASF1, X1 RX-2, X10 J1, X2 TX-2, X3 RESETJMP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

Commit message: up
Parts:
- removed R8, R9: 0, rcl:R1206
- added TP3: TPB1,27, testpad:B1,27
- moved X3 77.0 mm to (75.7, -0.13), turned to 180 degrees
- moved S4 75.5 mm to (85.0, 2.82)
- moved IC4 53.2 mm to (84.0, 69.6)
- moved S3 45.0 mm to (83.7, 46.7)
- moved SV1 37.6 mm to (101.0, 69.0)
- moved X9 32.2 mm to (21.7, -10.8)
- moved RS232-1 31.3 mm to (78.8, -12.0)
- moved X8 30.5 mm to (8.99, 80.7)
- moved RS-232-2 29.9 mm to (89.9, -12.1)
- moved LED3 27.1 mm to (83.7, 79.8)
- moved D1 26.5 mm to (65.7, -2.01), turned to 180 degrees
- moved SV2 26.0 mm to (84.3, 86.0), turned to 180 degrees
- moved POWER 13.6 mm to (65.2, -12.0)
- moved F1 12.6 mm to (83.8, 23.3)
- moved C3 12.3 mm to (33.5, 55.8), turned to 0 degrees
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Connections:
- removed net N$71: C11.1, C12.1, D1.C, F1.1
- new net RAW_VDD: F1.2, POWER.2, TP3.TP, X10.2
- net GND: no longer R9.1
- net VCC: no longer R8.1
- net VDD: now also C11.1, C12.1, D1.C, F1.1; no longer F1.2, POWER.2, R8.2, X10.2
- net VSS: no longer R9.2
Routing:
- net N$21: track 8.17 -> 81.0 mm, vias 0 -> 1
- net RAW_VDD: track 0.00 -> 71.2 mm, vias 0 -> 2
- net N$71: track 64.4 -> 0.00 mm, vias 1 -> 0
- net N$59: track 34.2 -> 92.0 mm, vias 1 -> 2
- net N$44: track 67.2 -> 123.4 mm, vias 1 -> 0
- net N$49: track 53.9 -> 108.4 mm, vias 1 -> 2
- net N$6: track 46.1 -> 100.3 mm, vias 1 -> 2
- net N$8: track 48.9 -> 99.8 mm
- net N$17: track 14.9 -> 65.7 mm
- net VDD: track 298.8 -> 349.2 mm, vias 6 -> 10
- net N$56: track 51.9 -> 101.3 mm
- net N$63: track 4.40 -> 53.6 mm, vias 0 -> 1
- net N$7: track 41.3 -> 90.2 mm, vias 1 -> 2
- net N$55: track 3.88 -> 51.4 mm, vias 0 -> 1
- net N$57: track 46.3 -> 0.00 mm, vias 1 -> 0
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Other:
- board text removed: "/fred/Downloads/mchp.bmp"

Commit message: up
Parts:
- added JMP1: 0R-JUMPA, jump-0r-smd:A0R-JMP
- added SV4: USB_TTL, con-lstb:MA06-1
- added X11: 22-23-2021, con-molex:22-23-2021
- moved R3 21.4 mm to (36.3, 43.2)
- moved C2 19.2 mm to (47.6, 57.0), flipped to the bottom, turned to 90 degrees
- moved F1 14.5 mm to (86.3, 37.6)
- moved C3 11.4 mm to (44.8, 57.1), flipped to the bottom, turned to 90 degrees
- moved C13 10.5 mm to (55.7, 49.5), flipped to the bottom, turned to 0 degrees
- moved C7 5.42 mm to (67.3, 54.3), flipped to the bottom, turned to 0 degrees
- moved R4 4.70 mm to (33.5, 47.9)
- moved C4 3.38 mm to (33.7, 51.7)
- moved C9 2.90 mm to (67.3, 59.4), flipped to the bottom
- moved R2 2.33 mm to (54.0, 43.2)
- moved IC1 2.31 mm to (46.2, 57.0)
- moved C16 1.42 mm to (72.2, 51.0)
- moved C21 0.81 mm to (54.1, 37.4)
- moved R6 0.28 mm to (41.8, 32.4)
- moved C1 0.18 mm to (48.3, 37.4), flipped to the bottom
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Connections:
- new net N$71: SV4.6, X11.2
- new net N$72: SV4.2, X11.1
- net GND: no longer C21.2, C7.2, JMP2.2, Q1.2
- net N$18: now also SV4.5
- net N$20: now also SV4.4
- net VCC: no longer JMP3.2
- net VDD: now also JMP3.2, JMP3.3, SV4.3
- net VSS: now also C21.2, C7.2, JMP1.1, JMP1.2, JMP1.3, JMP2.2, JMP2.3, Q1.2, SV4.1
Routing:
- net VDD: track 349.2 -> 74.3 mm, vias 10 -> 8
- net VSS: track 98.0 -> 214.0 mm, vias 11 -> 2
- net N$20: track 50.4 -> 102.8 mm, vias 2 -> 1
- net N$52: track 118.9 -> 169.7 mm, vias 2 -> 1
- net N$57: track 0.00 -> 49.5 mm, vias 0 -> 1
- net GND: track 83.9 -> 38.0 mm, vias 4 -> 1
- net N$4: track 48.9 -> 90.7 mm, vias 2 -> 0
- net N$44: track 123.4 -> 87.2 mm, vias 0 -> 2
- net N$65: track 38.0 -> 61.3 mm
- net VCC: track 79.3 -> 56.6 mm
- net N$60: track 50.4 -> 73.0 mm, vias 1 -> 0
- net N$46: track 60.3 -> 82.9 mm
- net N$47: track 101.3 -> 121.1 mm
- net N$71: track 0.00 -> 19.5 mm
- net N$42: track 45.1 -> 26.8 mm, vias 0 -> 1
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- added copper zone on layer 15, net VDD

Commit message: up
Parts:
- added JP1, JP2: GND, pinhead:1X01
- added SV5: ANA JUMPER, con-lstb:MA06-1
- added TP4, TP5: TPB1,27, testpad:B1,27
- moved LED3 67.1 mm to (28.8, 41.4)
- moved SV2 66.3 mm to (30.0, 48.0)
- moved SPI 62.3 mm to (5.03, 44.3)
- moved SV4 52.0 mm to (32.1, 16.3)
- moved X8 48.8 mm to (-27.3, 48.1)
- moved IC4 40.2 mm to (84.7, 29.4)
- moved C11 38.9 mm to (60.6, -5.87), turned to 0 degrees
- moved S3 33.6 mm to (84.6, 13.1)
- moved X7 29.7 mm to (5.36, 2.54), turned to 180 degrees
- moved X2 28.3 mm to (22.5, 23.1)
- moved X1 27.6 mm to (22.3, 15.3)
- moved SV1 26.0 mm to (89.6, 45.6), turned to 180 degrees
- moved X5 25.3 mm to (5.31, 23.9), turned to 180 degrees
- moved C4 23.1 mm to (32.7, 28.7)
- moved R4 20.0 mm to (39.3, 28.7)
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Connections:
- new net N$73: TP4.TP, X10.4
- new net N$74: TP5.TP, X10.6
- new net N$76: SV5.1, X9.6
- new net N$77: SV5.2, X9.7
- new net N$79: SV5.3, X9.11
- new net N$80: SV5.4, X9.12
- new net N$81: SV5.5, X9.13
- net N$54: now also X9.1
- net N$66: now also X9.2
- net RAW_VDD: now also X4.1
- net VDD: no longer X4.1
- net VSS: now also JP1.1, JP2.1, SV5.6, X9.5, X9.8
Routing:
- net VDD: track 74.3 -> 373.6 mm, vias 8 -> 6
- net N$52: track 169.7 -> 81.7 mm, vias 1 -> 3
- net N$76: track 0.00 -> 62.2 mm
- net N$54: track 65.9 -> 127.7 mm, vias 3 -> 1
- net N$77: track 0.00 -> 55.4 mm
- net N$66: track 59.0 -> 112.6 mm
- net N$39: track 127.8 -> 171.1 mm, vias 2 -> 1
- net N$29: track 17.5 -> 57.3 mm, vias 0 -> 1
- net N$31: track 18.5 -> 56.3 mm, vias 0 -> 1
- net N$79: track 0.00 -> 36.8 mm
- net N$35: track 77.3 -> 114.0 mm, vias 2 -> 1
- net N$20: track 102.8 -> 70.0 mm, vias 1 -> 2
- net N$74: track 0.00 -> 32.8 mm
- net N$32: track 28.0 -> 60.4 mm, vias 0 -> 1
- net N$30: track 23.0 -> 54.9 mm, vias 0 -> 2
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- removed copper zone on layer 15, net VDD
Other:
- board size 130.5 x 111.1 mm -> 152.6 x 75 mm

Commit message: up
Parts:
- added LED1: 5v, led:CHIPLED_1206
- added LED2: -15, led:CHIPLED_1206
- added LED4: +15, led:CHIPLED_1206
- added R13, R9: 3K, rcl:R1206
- added R8: 1K, rcl:R1206
- moved F1 10.9 mm to (81.5, 21.2)
Connections:
- removed net N$73: TP4.TP, X10.4
- removed net N$74: TP5.TP, X10.6
- new net N$75: LED1.A, R8.2
- new net N$78: LED2.C, R9.2
- new net N$82: LED4.A, R13.2
- new net N15V: R9.1, TP5.TP, X10.6
- new net P15V: R13.1, TP4.TP, X10.4
- net GND: now also JMP2.2
- net RAW_VDD: now also R8.1
- net VCC: now also JMP3.2
- net VDD: no longer JMP3.2
- net VSS: now also LED1.C, LED2.A, LED4.C; no longer JMP2.2
Routing:
- net VSS: track 233.0 -> 300.3 mm, vias 3 -> 2
- net N15V: track 0.00 -> 57.3 mm
- net P15V: track 0.00 -> 40.9 mm
- net N$36: track 107.3 -> 147.6 mm
- net N$74: track 32.8 -> 0.00 mm
- net N$56: track 81.7 -> 58.6 mm, vias 1 -> 3
- net N$40: track 100.1 -> 123.2 mm, vias 1 -> 2
- net N$4: track 80.1 -> 102.4 mm
- net N$20: track 70.0 -> 90.8 mm, vias 2 -> 0
- net N$73: track 19.5 -> 0.00 mm
- net N$58: track 80.3 -> 99.5 mm, vias 3 -> 2
- net VCC: track 52.8 -> 69.5 mm, vias 2 -> 4
- net N$53: track 69.9 -> 53.3 mm, vias 0 -> 2
- net N$21: track 70.0 -> 54.7 mm, vias 0 -> 1
- net N$13: track 34.6 -> 19.5 mm, vias 0 -> 1
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Other:
- board text added: "1.9 FGB@MCHP PS CONTROLLER"
- board text removed: "1.8 FGB@MCHP PS CONTROLLER"

Commit message: up
Parts:
- removed JMP1: 0R-JUMPA, jump-0r-smd:A0R-JMP
- added VSS-GND-1: 0R-JUMPA, jump-0r-smd:A0R-JMP
- R1: value 220 -> 56
- R11, R4, R7: value 220 -> 1k
- VDD-VCC: value 0R-JUMPA -> VDD-VCC
- VSS-GND: value 0R-JUMPA -> VSS-GND
- renumbered JMP2 to VSS-GND, JMP3 to VDD-VCC, SV1 to ICSP
Connections:
- net N$1 renamed VPP
- net N$4 renamed CPUCLK
- net N$6 renamed PGD
- net N$7 renamed PGC
- net N$8 renamed ADCREF
- net GND: now also VSS-GND-1.3
- net VDD: now also RS-232-2.4, RS232-1.4
- net VSS: now also VSS-GND-1.1, VSS-GND-1.2; no longer JMP1.1, JMP1.2, JMP1.3
Routing:
- net VDD: track 364.2 -> 401.1 mm, vias 9 -> 10
- net GND: track 48.9 -> 54.5 mm
Other:
- board text added: "V"

Commit message: up
Parts:
- added ANAO0: PS V, jump-0r-smd:A0R-JMP
- added ANAO1: PS I, jump-0r-smd:A0R-JMP
- added C10, C8: 1uf, rcl:C0805
- added L1, L2: 1K, rcl:L2012C
- moved LED3 56.0 mm to (84.6, 38.5)
Connections:
- removed net N$44: IC1.44, X6.2
- removed net N$50: IC1.38, X6.9
- new net DACOUT: ANAO0.3, ANAO1.3, IC1.23, X5.2
- new net N$1: C8.1, L1.2, X9.9
- new net N$4: C10.1, L2.2, X9.10
- new net N$8: ANAO0.2, L1.1
- new net PWM5: ANAO0.1, IC1.38, X6.10
- new net PWM6: ANAO1.1, IC1.44, X6.2
- net N$37: now also ANAO1.2, L2.1; no longer IC1.23, X5.2, X9.10, X9.9
- net VSS: now also C10.2, C8.2, X6.9; no longer X6.10
Routing:
- net PWM6: track 0.00 -> 105.5 mm, vias 0 -> 2
- net DACOUT: track 0.00 -> 100.0 mm, vias 0 -> 2
- net PWM5: track 0.00 -> 97.2 mm, vias 0 -> 1
- net N$50: track 76.1 -> 0.00 mm, vias 1 -> 0
- net N$37: track 88.9 -> 24.3 mm, vias 2 -> 0
- net N$44: track 59.6 -> 0.00 mm, vias 2 -> 0
- net N$65: track 62.5 -> 11.1 mm, vias 2 -> 0
- net N$39: track 159.5 -> 202.4 mm
- net N$1: track 0.00 -> 35.1 mm
- net N$36: track 147.6 -> 114.3 mm
- net N$55: track 57.1 -> 88.5 mm
- net N$4: track 0.00 -> 24.6 mm
- net N$25: track 61.3 -> 86.0 mm
- net N$35: track 120.7 -> 96.7 mm, vias 1 -> 3
- net N$45: track 63.2 -> 86.2 mm
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