File: pic_k42.brd (EAGLE design)
At the start: 152.6 x 75 mm, 82 parts, among them IC1 PIC18F57K42-E_PT, IC2 REF3440IDBVR, IC3 MAX232, IC4 ILAMP, K1 G6K-2P, Q1 ASF1, X1 RX-2, X10 J1, X11 22-23-2021, X2 TX-2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

Commit message: up
Parts:
- moved X4 132.4 mm to (-30.3, -14.0), turned to 90 degrees
- moved SV3 69.4 mm to (27.1, 12.4)
- moved JP2 53.7 mm to (102.5, -16.1)
- moved TP5 9.97 mm to (91.9, 39.8)
- moved TP4 9.34 mm to (92.2, 35.5)
Connections:
- net N$37 renamed ANAS1
- net N$76 renamed ANAJ1
- net N$77 renamed ANAJ2
- net N$79 renamed ANAJ3
- net N$8 renamed ANAS0
- net N$80 renamed ANAJ4
- net N$81 renamed ANAJ5
- removed net N$1: C8.1, L1.2, X9.9
- removed net N$24: IC1.28, SV2.3
- removed net N$4: C10.1, L2.2, X9.10
- removed net N$41: IC1.36, SPI.9
- removed net N$42: IC1.37, SPI.10
- new net OUT0FIL: C8.1, IC1.36, L1.2, SPI.9, X9.9
- new net OUT1FIL: C10.1, IC1.37, L2.2, SPI.10, X9.10
- net DACOUT: now also IC1.28, SV2.3
Routing:
- net OUT0FIL: track 0.00 -> 129.7 mm, vias 0 -> 2
- net OUT1FIL: track 0.00 -> 126.3 mm, vias 0 -> 3
- net RAW_VDD: track 89.7 -> 201.8 mm, vias 0 -> 2
- net N$39: track 202.4 -> 130.2 mm, vias 1 -> 4
- net N$67: track 7.38 -> 77.2 mm
- net N$69: track 5.68 -> 70.5 mm
- net N$68: track 6.41 -> 69.8 mm, vias 0 -> 1
- net DACOUT: track 100.0 -> 149.8 mm, vias 2 -> 4
- net N$41: track 42.2 -> 0.00 mm, vias 1 -> 0
- net N$42: track 38.7 -> 0.00 mm, vias 2 -> 0
- net VDD: track 398.5 -> 436.0 mm, vias 9 -> 8
- net N$55: track 88.5 -> 51.9 mm, vias 2 -> 1
- net N$1: track 35.1 -> 0.00 mm
- net N$24: track 27.2 -> 0.00 mm
- net N$4: track 24.6 -> 0.00 mm
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
Commit message: up
Parts:
- added C22: 0.1, rcl:C1206
- added C23: 1uf, rcl:C0805
- added P10_V: 10 volts, con-lstb:MA03-1
- added U1: LM78L05ACMX/NOPB, LM78L05ACMX_NOPB:SOIC127P599X175-8N
- added VI_OUT_JUMPER: out jumper, con-lstb:MA03-1
- moved R6 37.7 mm to (72.8, 39.6), turned to 0 degrees
- moved R3 35.7 mm to (72.9, 24.1)
- moved R5 32.7 mm to (72.9, 34.3)
- moved R11 14.8 mm to (84.8, 41.5)
- moved R2 11.0 mm to (48.3, 23.3)
- moved SPI 5.44 mm to (4.27, 49.7)
- moved C15 3.46 mm to (62.3, 29.2)
- moved IC2 3.28 mm to (62.3, 34.0)
- moved Q1 3.02 mm to (62.6, 43.1)
- moved ICSP 2.45 mm to (88.6, 47.8)
- moved SV2 2.12 mm to (29.0, 49.9)
- moved C16 0.79 mm to (72.8, 44.5)
- moved R12 0.24 mm to (72.8, 29.1)
- moved R1 0.20 mm to (47.0, 28.6)
Connections:
- new net NC_4: U1.4
- new net NC_5: U1.5
- new net P10V: C22.1, P10_V.1, P10_V.2, U1.1
- net OUT0FIL: now also VI_OUT_JUMPER.1
- net OUT1FIL: now also VI_OUT_JUMPER.2
- net P15V: now also C23.1, U1.8
- net VSS: now also C22.2, C23.2, P10_V.3, U1.2, U1.3, U1.6, U1.7, VI_OUT_JUMPER.3
Routing:
- net P15V: track 41.9 -> 222.0 mm, vias 0 -> 2
- net OUT0FIL: track 129.7 -> 192.3 mm, vias 2 -> 4
- net OUT1FIL: track 126.3 -> 176.4 mm
- net N$17: track 55.2 -> 17.0 mm, vias 1 -> 0
- net N$55: track 51.9 -> 14.8 mm, vias 1 -> 0
- net DACOUT: track 149.8 -> 112.7 mm, vias 4 -> 5
- net N$3: track 41.5 -> 7.00 mm, vias 1 -> 0
- net N$36: track 138.2 -> 104.9 mm, vias 1 -> 5
- net N$61: track 12.8 -> 40.8 mm, vias 0 -> 2
- net VDD: track 436.0 -> 408.3 mm
- net N$46: track 70.0 -> 97.4 mm
- net N$53: track 51.6 -> 75.2 mm, vias 2 -> 0
- net N$45: track 75.7 -> 54.0 mm
- net N$70: track 77.6 -> 99.0 mm
- net PWM5: track 109.4 -> 89.7 mm
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Other:
- board text added: "2.0 FGB@MCHP PS CONTROLLER"
- board text removed: "1.9 FGB@MCHP PS CONTROLLER"

Commit message: up
Parts:
- added J1: MLE-105-01-G-DV, MLE-105-01-G-DV:SAMTEC_MLE-105-01-G-DV
Changed lines of the file:
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@@
 <attribute name="VALUE" x="-31.9532" y="7.3406" size="1.27" layer="27" ratio="10"/>
+</element>
+<element name="J1" library="MLE-105-01-G-DV" package="SAMTEC_MLE-105-01-G-DV" value="MLE-105-01-G-DV" x="-30.9372" y="32.3342" smashed="yes" rot="R90">
+<attribute name="MANUFACTURER" value="SAMTEC " x="-30.9372" y="32.3342" size="1.778" layer="27" rot="R90" display="off"/>
+<attribute name="NAME" x="-34.4922" y="28.7342" size="1.27" layer="25" rot="R90"/>
+<attribute name="VALUE" x="-26.1322" y="28.7342" size="1.27" layer="27" rot="R90"/>
 </element>
 </elements>

Commit message: up
Parts:
- R12: value 220 -> 56
- R13, R9: value 3K -> 3.83K
Changed lines of the file:
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@@
 <attribute name="VALUE" x="71.0946" y="6.7564" size="0.0254" layer="27"/>
 </element>
-<element name="R12" library="rcl" library_urn="urn:adsk.eagle:library:334" package="R1206" package3d_urn="urn:adsk.eagle:package:23540/2" value="220" x="72.8472" y="29.1084" smashed="yes">
+<element name="R12" library="rcl" library_urn="urn:adsk.eagle:library:334" package="R1206" package3d_urn="urn:adsk.eagle:package:23540/2" value="56" x="72.8472" y="29.1084" smashed="yes">
 <attribute name="NAME" x="71.5772" y="30.3784" size="1.27" layer="25"/>
 <attribute name="SPICEPREFIX" value="R" x="72.8472" y="29.1084" size="1.778" layer="27" display="off"/>
@@
 <attribute name="VALUE" x="96.4438" y="13.5128" size="1.27" layer="27" rot="R90"/>
 </element>
-<element name="R9" library="rcl" library_urn="urn:adsk.eagle:library:334" package="R1206" package3d_urn="urn:adsk.eagle:package:23540/2" value="3K" x="82.0928" y="5.5626" smashed="yes">
+<element name="R9" library="rcl" library_urn="urn:adsk.eagle:library:334" package="R1206" package3d_urn="urn:adsk.eagle:package:23540/2" value="3.83K" x="82.0928" y="5.5626" smashed="yes">
 <attribute name="NAME" x="80.8228" y="6.8326" size="1.27" layer="25"/>
 <attribute name="SPICEPREFIX" value="R" x="82.0928" y="5.5626" size="1.778" layer="27" display="off"/>
 <attribute name="VALUE" x="80.8228" y="3.0226" size="1.27" layer="27"/>
 </element>
-<element name="R13" library="rcl" library_urn="urn:adsk.eagle:library:334" package="R1206" package3d_urn="urn:adsk.eagle:package:23540/2" value="3K" x="88.265" y="5.4356" smashed="yes">
+<element name="R13" library="rcl" library_urn="urn:adsk.eagle:library:334" package="R1206" package3d_urn="urn:adsk.eagle:package:23540/2" value="3.83K" x="88.265" y="5.4356" smashed="yes">
 <attribute name="NAME" x="86.995" y="6.7056" size="1.27" layer="25"/>
 <attribute name="SPICEPREFIX" value="R" x="88.265" y="5.4356" size="1.778" layer="27" display="off"/>

Commit message: up
Connections:
- net N$30 renamed SDO1
- net N$31 renamed SCK1
- net N$33 renamed CSB
Changed lines of the file:
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@@
 <via x="44.2722" y="48.6156" extent="1-16" drill="0.35"/>
 </signal>
-<signal name="N$30">
+<signal name="SDO1">
 <contactref element="SPI" pad="2"/>
 <contactref element="IC1" pad="47"/>
@@
 <via x="6.0198" y="51.816" extent="1-16" drill="0.35"/>
 </signal>
-<signal name="N$31">
+<signal name="SCK1">
 <contactref element="SPI" pad="3"/>
 <contactref element="IC1" pad="41"/>
@@
 <via x="49.6824" y="52.2732" extent="1-16" drill="0.35"/>
 </signal>
-<signal name="N$33">
+<signal name="CSB">
 <contactref element="SPI" pad="5"/>
 <contactref element="IC1" pad="40"/>

Commit message: Revert "up"
This reverts commit 2af174bc1ac14fa5ed8294ec6c26e2dbc3c0e6fd.
Connections:
- net CSB renamed N$33
- net SCK1 renamed N$31
- net SDO1 renamed N$30
Changed lines of the file:
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@@
 <via x="44.2722" y="48.6156" extent="1-16" drill="0.35"/>
 </signal>
-<signal name="SDO1">
+<signal name="N$30">
 <contactref element="SPI" pad="2"/>
 <contactref element="IC1" pad="47"/>
@@
 <via x="6.0198" y="51.816" extent="1-16" drill="0.35"/>
 </signal>
-<signal name="SCK1">
+<signal name="N$31">
 <contactref element="SPI" pad="3"/>
 <contactref element="IC1" pad="41"/>
@@
 <via x="49.6824" y="52.2732" extent="1-16" drill="0.35"/>
 </signal>
-<signal name="CSB">
+<signal name="N$33">
 <contactref element="SPI" pad="5"/>
 <contactref element="IC1" pad="40"/>

Commit message: up
Connections:
- net N$38 renamed RA1
- net N$39 renamed RA0
- net N$54 renamed ANRB2
- net N$66 renamed ANRB3
Changed lines of the file:
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@@
 <param name="tpViaShape" value="round"/>
 <param name="PrefDir.1" value="a"/>
-<param name="PrefDir.2" value="a"/>
+<param name="PrefDir.2" value="0"/>
 <param name="PrefDir.3" value="0"/>
 <param name="PrefDir.4" value="0"/>
@@
 <param name="PrefDir.13" value="0"/>
 <param name="PrefDir.14" value="0"/>
-<param name="PrefDir.15" value="a"/>
+<param name="PrefDir.15" value="0"/>
 <param name="PrefDir.16" value="a"/>
 <param name="cfVia" value="90"/>
@@
 <via x="28.4226" y="45.7962" extent="1-16" drill="0.35"/>
 </signal>
-<signal name="N$38">
+<signal name="RA1">
 <contactref element="X5" pad="1"/>
 <contactref element="IC1" pad="22"/>
@@
 <via x="19.2786" y="21.336" extent="1-16" drill="0.35"/>
 </signal>
-<signal name="N$39">
+<signal name="RA0">
 <contactref element="X5" pad="10"/>
 <contactref element="IC1" pad="21"/>
@@
 <wire x1="43.5102" y1="42.291" x2="43.5394" y2="42.2602" width="0.1524" layer="1"/>
 </signal>
-<signal name="N$54">
+<signal name="ANRB2">
 <contactref element="X7" pad="2"/>
 <contactref element="IC1" pad="10"/>
@@
 <via x="57.912" y="9.144" extent="1-16" drill="0.35"/>
 </signal>
-<signal name="N$66">
+<signal name="ANRB3">
 <contactref element="X7" pad="3"/>
 <contactref element="IC1" pad="11"/>
