File: pic_k42.sch (EAGLE design)
At the start: 62 parts, among them IC1 PIC18F57K42-E_PT, IC2 REF3440IDBVR, IC3 MAX232, IC4 ILAMP, K1 G6K-2P, Q1 ASF1, X1 RX-2, X10 J1, X2 TX-2, X3 RESETJMP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

Commit message: up
Parts:
- added JMP1: 0R-JUMPA, jump-0r-smd:0R-JUMPA
- added SV4: USB_TTL, con-lstb:MA06-1
- added X11: 22-23-2021, con-molex:22-23-2021
Connections:
- new net N$71: SV4.6, X11-2.S
- new net N$72: SV4.2, X11-1.S
- net GND: no longer C21.2, C7.2, JMP2-0R.2, Q1.GND
- net N$18: now also SV4.5
- net N$20: now also SV4.4
- net VCC: no longer JMP3-0R.2
- net VDD: now also JMP3-0R.2, JMP3-0R.3, SV4.3
- net VSS: now also C21.2, C7.2, JMP1-0R.1, JMP1-0R.2, JMP1-0R.3, JMP2-0R.2, JMP2-0R.3, Q1.GND, SV4.1

Commit message: up
Parts:
- added JP1, JP2: GND, pinhead:PINHD-1X1
- added SV5: ANA JUMPER, con-lstb:MA06-1
- added TP4, TP5: TPB1,27, testpad:TPB1,27
Connections:
- new net N$73: TP4.TP, X10-4.S
- new net N$74: TP5.TP, X10-6.S
- new net N$76: SV5.1, X9-6.S
- new net N$77: SV5.2, X9-7.S
- new net N$79: SV5.3, X9-11.S
- new net N$80: SV5.4, X9-12.S
- new net N$81: SV5.5, X9-13.S
- net N$54: now also X9-1.S
- net N$66: now also X9-2.S
- net RAW_VDD: now also X4.1
- net VDD: no longer X4.1
- net VSS: now also JP1.1, JP2.1, SV5.6, X9-5.S, X9-8.S

Commit message: up
Parts:
- added LED1: 5v, led:LEDCHIPLED_1206
- added LED2: -15, led:LEDCHIPLED_1206
- added LED4: +15, led:LEDCHIPLED_1206
- added R13, R9: 3K, rcl:R-US_R1206
- added R8: 1K, rcl:R-US_R1206
Connections:
- removed net N$73: TP4.TP, X10-4.S
- removed net N$74: TP5.TP, X10-6.S
- new net N$75: LED1.A, R8.2
- new net N$78: LED2.C, R9.2
- new net N$82: LED4.A, R13.2
- new net N15V: R9.1, TP5.TP, X10-6.S
- new net P15V: R13.1, TP4.TP, X10-4.S
- net GND: now also JMP2-0R.2
- net RAW_VDD: now also R8.1
- net VCC: now also JMP3-0R.2
- net VDD: no longer JMP3-0R.2
- net VSS: now also LED1.C, LED2.A, LED4.C; no longer JMP2-0R.2
Other:
- moved on the sheet: TP4, TP5

Commit message: up
Parts:
- R1: value 220 -> 56
- R11, R4, R7: value 220 -> 1k
- VDD-VCC: value 0R-JUMPA -> VDD-VCC
- VSS-GND: value 0R-JUMPA -> VSS-GND
- renumbered JMP1 to VSS-GND-1, JMP2 to VSS-GND, JMP3 to VDD-VCC, SV1 to ICSP
Connections:
- net N$1 renamed VPP
- net N$4 renamed CPUCLK
- net N$6 renamed PGD
- net N$7 renamed PGC
- net N$8 renamed ADCREF
- net GND: now also VSS-GND-1-0R.3
- net VDD: now also RS-232-2.4, RS232-1.4
- net VSS: no longer VSS-GND-1-0R.3
Other:
- note added: "V"

Commit message: up
Parts:
- added ANAO0: PS V, jump-0r-smd:0R-JUMPA
- added ANAO1: PS I, jump-0r-smd:0R-JUMPA
- added C10, C8: 1uf, rcl:C-USC0805
- added L1, L2: 1K, rcl:L-USL2012C
Connections:
- removed net N$44: IC1.RD2, X6-2.S
- removed net N$50: IC1.RF2, X6-9.S
- new net DACOUT: ANAO0-0R.3, ANAO1-0R.3, IC1.RA2, X5-2.S
- new net N$1: C8.1, L1.2, X9-9.S
- new net N$4: C10.1, L2.2, X9-10.S
- new net N$8: ANAO0-0R.2, L1.1
- new net PWM5: ANAO0-0R.1, IC1.RF2, X6-10.S
- new net PWM6: ANAO1-0R.1, IC1.RD2, X6-2.S
- net N$37: now also ANAO1-0R.2, L2.1; no longer IC1.RA2, X5-2.S, X9-10.S, X9-9.S
- net VSS: now also C10.2, C8.2, X6-9.S; no longer X6-10.S

Commit message: up
Connections:
- net N$37 renamed ANAS1
- net N$76 renamed ANAJ1
- net N$77 renamed ANAJ2
- net N$79 renamed ANAJ3
- net N$8 renamed ANAS0
- net N$80 renamed ANAJ4
- net N$81 renamed ANAJ5
- removed net N$1: C8.1, L1.2, X9-9.S
- removed net N$24: IC1.RE1, SV2.3
- removed net N$4: C10.1, L2.2, X9-10.S
- removed net N$41: IC1.RF0, SPI-9.S
- removed net N$42: IC1.RF1, SPI-10.S
- new net OUT0FIL: C8.1, IC1.RF0, L1.2, SPI-9.S, X9-9.S
- new net OUT1FIL: C10.1, IC1.RF1, L2.2, SPI-10.S, X9-10.S
- net DACOUT: now also IC1.RE1, SV2.3

Commit message: up
Parts:
- added C22: 0.1, rcl:C-USC1206
- added C23: 1uf, rcl:C-USC0805
- added P10_V: 10 volts, con-lstb:MA03-1
- added U1: LM78L05ACMX/NOPB, LM78L05ACMX_NOPB:LM78L05ACMX/NOPB
- added VI_OUT_JUMPER: out jumper, con-lstb:MA03-1
Connections:
- new net P10V: C22.1, P10_V.1, P10_V.2, U1.VOUT
- net OUT0FIL: now also VI_OUT_JUMPER.1
- net OUT1FIL: now also VI_OUT_JUMPER.2
- net P15V: now also C23.1, U1.VIN
- net VSS: now also C22.2, C23.2, P10_V.3, U1.GND_2, U1.GND_3, U1.GND_6, U1.GND_7, VI_OUT_JUMPER.3
Changed lines of the file:
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@@
 <part name="VSS55" library="supply1" library_urn="urn:adsk.eagle:library:371" deviceset="VSS" device=""/>
 <part name="VSS56" library="supply1" library_urn="urn:adsk.eagle:library:371" deviceset="VSS" device=""/>
+<part name="U1" library="LM78L05ACMX_NOPB" deviceset="LM78L05ACMX/NOPB" device=""/>
+<part name="VSS12" library="supply1" library_urn="urn:adsk.eagle:library:371" deviceset="VSS" device=""/>
+<part name="C22" library="rcl" library_urn="urn:adsk.eagle:library:334" deviceset="C-US" device="C1206" package3d_urn="urn:adsk.eagle:package:23618/2" value="0.1"/>
+<part name="VSS57" library="supply1" library_urn="urn:adsk.eagle:library:371" deviceset="VSS" device=""/>
+<part name="C23" library="rcl" library_urn="urn:adsk.eagle:library:334" deviceset="C-US" device="C0805" package3d_urn="urn:adsk.eagle:package:23617/2" value="1uf"/>
+<part name="VSS58" library="supply1" library_urn="urn:adsk.eagle:library:371" deviceset="VSS" device=""/>
+<part name="P10_V" library="con-lstb" library_urn="urn:adsk.eagle:library:162" deviceset="MA03-1" device="" package3d_urn="urn:adsk.eagle:package:8339/1" value="10 volts"/>
+<part name="VI_OUT_JUMPER" library="con-lstb" library_urn="urn:adsk.eagle:library:162" deviceset="MA03-1" device="" package3d_urn="urn:adsk.eagle:package:8339/1" value="out jumper"/>
+<part name="VSS59" library="supply1" library_urn="urn:adsk.eagle:library:371" deviceset="VSS" device=""/>
+<part name="VSS60" library="supply1" library_urn="urn:adsk.eagle:library:371" deviceset="VSS" device=""/>
 </parts>
 <sheets>
@@
 <attribute name="NAME" x="-203.2" y="16.51" size="1.778" layer="95"/>
 </instance>
-<instance part="ANAO0" gate="G$2" x="-177.8" y="66.04" smashed="yes"/>
+<instance part="ANAO0" gate="G$2" x="-208.28" y="17.78" smashed="yes"/>
 <instance part="ANAO1" gate="-0R" x="-205.74" y="7.62" smashed="yes">
 <attribute name="NAME" x="-203.2" y="8.89" size="1.778" layer="95"/>
@@
 <instance part="VSS56" gate="G$1" x="-30.48" y="86.36" smashed="yes" rot="R180">
 <attribute name="VALUE" x="-27.94" y="91.44" size="1.778" layer="96" rot="R270"/>
+</instance>
+<instance part="U1" gate="G$1" x="-187.96" y="93.98" smashed="yes">
+<attribute name="NAME" x="-200.66" y="107.68" size="2.0828" layer="95" ratio="10" rot="SR0"/>
+<attribute name="VALUE" x="-200.66" y="77.28" size="2.0828" layer="96" ratio="10" rot="SR0"/>
+</instance>
+<instance part="VSS12" gate="G$1" x="-167.64" y="96.52" smashed="yes" rot="R90">
+<attribute name="VALUE" x="-162.56" y="93.98" size="1.778" layer="96" rot="R180"/>
+</instance>
+<instance part="C22" gate="G$1" x="-157.48" y="101.6" smashed="yes">
+<attribute name="NAME" x="-156.464" y="102.235" size="1.778" layer="95"/>
+<attribute name="VALUE" x="-156.464" y="97.409" size="1.778" layer="96"/>
+</instance>
+<instance part="VSS57" gate="G$1" x="-157.48" y="93.98" smashed="yes">
+<attribute name="VALUE" x="-160.02" y="88.9" size="1.778" layer="96" rot="R90"/>
+</instance>
+<instance part="C23" gate="G$1" x="-213.36" y="101.6" smashed="yes">
+<attribute name="NAME" x="-222.504" y="99.695" size="1.778" layer="95"/>
+<attribute name="VALUE" x="-212.344" y="97.409" size="1.778" layer="96"/>
+</instance>
+<instance part="VSS58" gate="G$1" x="-213.36" y="93.98" smashed="yes">
+<attribute name="VALUE" x="-215.9" y="88.9" size="1.778" layer="96" rot="R90"/>
+</instance>
+<instance part="P10_V" gate="G$1" x="-139.7" y="104.14" smashed="yes" rot="R180">
+<attribute name="VALUE" x="-138.43" y="111.76" size="1.778" layer="96" rot="R180"/>
+<attribute name="NAME" x="-138.43" y="98.298" size="1.778" layer="95" rot="R180"/>
+</instance>
+<instance part="VI_OUT_JUMPER" gate="G$1" x="-139.7" y="73.66" smashed="yes" rot="R180">
+<attribute name="VALUE" x="-138.43" y="81.28" size="1.778" layer="96" rot="R180"/>
+<attribute name="NAME" x="-135.89" y="65.278" size="1.778" layer="95" rot="R180"/>
+</instance>
+<instance part="VSS59" gate="G$1" x="-147.32" y="68.58" smashed="yes">
+<attribute name="VALUE" x="-152.4" y="71.12" size="1.778" layer="96" rot="R180"/>
+</instance>
+<instance part="VSS60" gate="G$1" x="-147.32" y="99.06" smashed="yes">
+<attribute name="VALUE" x="-147.32" y="96.52" size="1.778" layer="96" rot="R180"/>
 </instance>
 </instances>
@@
 <pinref part="VDD12" gate="G$1" pin="VDD"/>
 <junction x="-172.72" y="55.88"/>
+<junction x="-180.34" y="55.88"/>
 </segment>
 <segment>
@@
 <pinref part="VSS35" gate="G$1" pin="VSS"/>
 <junction x="-172.72" y="45.72"/>
+<junction x="-177.8" y="45.72"/>
 </segment>
 <segment>
@@
 <wire x1="-30.48" y1="83.82" x2="-33.02" y2="83.82" width="0.1524" layer="91"/>
 <junction x="-33.02" y="83.82"/>
+</segment>
+<segment>
+<pinref part="U1" gate="G$1" pin="GND_6"/>
+<pinref part="U1" gate="G$1" pin="GND_7"/>
+<wire x1="-170.18" y1="93.98" x2="-170.18" y2="91.44" width="0.1524" layer="91"/>
+<pinref part="U1" gate="G$1" pin="GND_2"/>
+<pinref part="U1" gate="G$1" pin="GND_3"/>
+<wire x1="-170.18" y1="99.06" x2="-170.18" y2="96.52" width="0.1524" layer="91"/>
+<wire x1="-170.18" y1="93.98" x2="-170.18" y2="96.52" width="0.1524" layer="91"/>
+<junction x="-170.18" y="93.98"/>
+<junction x="-170.18" y="96.52"/>
+<pinref part="VSS12" gate="G$1" pin="VSS"/>
+<junction x="-170.18" y="99.06"/>
+<junction x="-170.18" y="91.44"/>
+</segment>
+<segment>
+<pinref part="C22" gate="G$1" pin="2"/>
+<pinref part="VSS57" gate="G$1" pin="VSS"/>
+<junction x="-157.48" y="96.52"/>
+</segment>
+<segment>
+<pinref part="C23" gate="G$1" pin="2"/>
+<pinref part="VSS58" gate="G$1" pin="VSS"/>
+<junction x="-213.36" y="96.52"/>
+</segment>
+<segment>
+<pinref part="VI_OUT_JUMPER" gate="G$1" pin="3"/>
+<pinref part="VSS59" gate="G$1" pin="VSS"/>
+<junction x="-147.32" y="71.12"/>
+</segment>
+<segment>
+<pinref part="P10_V" gate="G$1" pin="3"/>
+<pinref part="VSS60" gate="G$1" pin="VSS"/>
+<junction x="-147.32" y="101.6"/>
 </segment>
 </net>
@@
 <junction x="-177.8" y="-35.56"/>
 <junction x="-170.18" y="-35.56"/>
-<label x="-193.04" y="-35.56" size="1.778" layer="95" rot="R180"/>
+<label x="-172.72" y="-35.56" size="1.778" layer="95" rot="R180"/>
 </segment>
 <segment>
 <wire x1="-177.8" y1="-43.18" x2="-185.42" y2="-43.18" width="0.1524" layer="91"/>
 <pinref part="R13" gate="G$1" pin="1"/>
-<label x="-177.8" y="-50.8" size="1.778" layer="95" rot="R180"/>
+<label x="-182.88" y="-40.64" size="1.778" layer="95" rot="R180"/>
 <junction x="-185.42" y="-43.18"/>
+</segment>
+<segment>
+<wire x1="-205.74" y1="104.14" x2="-213.36" y2="104.14" width="0.1524" layer="91"/>
+<pinref part="U1" gate="G$1" pin="VIN"/>
+<pinref part="C23" gate="G$1" pin="1"/>
+<junction x="-213.36" y="104.14"/>
+<junction x="-205.74" y="104.14"/>
+<label x="-220.98" y="104.14" size="1.778" layer="95"/>
 </segment>
 </net>
@@
 <junction x="-175.26" y="-40.64"/>
 <junction x="-170.18" y="-40.64"/>
-<label x="-185.42" y="-40.64" size="1.778" layer="95" rot="R180"/>
+<label x="-170.18" y="-40.64" size="1.778" layer="95" rot="R180"/>
 </segment>
 <segment>
@@
 <junction x="106.68" y="91.44"/>
 </segment>
+<segment>
+<wire x1="-147.32" y1="73.66" x2="-154.94" y2="73.66" width="0.1524" layer="91"/>
+<pinref part="VI_OUT_JUMPER" gate="G$1" pin="2"/>
+<junction x="-147.32" y="73.66"/>
+<label x="-167.64" y="73.66" size="1.778" layer="95"/>
+</segment>
 </net>
 <net name="OUT0FIL" class="0">
@@
 <junction x="139.7" y="55.88"/>
 </segment>
-</net>
+<segment>
+<wire x1="-147.32" y1="76.2" x2="-154.94" y2="76.2" width="0.1524" layer="91"/>
+<pinref part="VI_OUT_JUMPER" gate="G$1" pin="1"/>
+<junction x="-147.32" y="76.2"/>
+<label x="-167.64" y="76.2" size="1.778" layer="95"/>
+</segment>
+</net>
+<net name="P10V" class="0">
+<segment>
+<pinref part="U1" gate="G$1" pin="VOUT"/>
+<wire x1="-170.18" y1="104.14" x2="-157.48" y2="104.14" width="0.1524" layer="91"/>
+<junction x="-170.18" y="104.14"/>
+<pinref part="C22" gate="G$1" pin="1"/>
+<wire x1="-157.48" y1="104.14" x2="-152.4" y2="104.14" width="0.1524" layer="91"/>
+<junction x="-157.48" y="104.14"/>
+<label x="-162.56" y="106.68" size="1.778" layer="95"/>
+<pinref part="P10_V" gate="G$1" pin="1"/>
+<wire x1="-147.32" y1="106.68" x2="-152.4" y2="106.68" width="0.1524" layer="91"/>
+<wire x1="-152.4" y1="106.68" x2="-152.4" y2="104.14" width="0.1524" layer="91"/>
+<pinref part="P10_V" gate="G$1" pin="2"/>
+<wire x1="-152.4" y1="104.14" x2="-147.32" y2="104.14" width="0.1524" layer="91"/>
+<junction x="-152.4" y="104.14"/>
+<junction x="-147.32" y="104.14"/>
+<junction x="-147.32" y="106.68"/>
+</segment>
+</net>

Commit message: up
Parts:
- added J1: MLE-105-01-G-DV, MLE-105-01-G-DV:MLE-105-01-G-DV
Changed lines of the file:
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@@
 <part name="VSS59" library="supply1" library_urn="urn:adsk.eagle:library:371" deviceset="VSS" device=""/>
 <part name="VSS60" library="supply1" library_urn="urn:adsk.eagle:library:371" deviceset="VSS" device=""/>
+<part name="J1" library="MLE-105-01-G-DV" deviceset="MLE-105-01-G-DV" device=""/>
 </parts>
 <sheets>
@@
 <attribute name="VALUE" x="-147.32" y="96.52" size="1.778" layer="96" rot="R180"/>
 </instance>
+<instance part="J1" gate="G$1" x="-220.98" y="38.1" smashed="yes">
+<attribute name="NAME" x="-229.1" y="46.836" size="1.778" layer="95"/>
+<attribute name="VALUE" x="-228.6" y="27.94" size="1.778" layer="96"/>
+</instance>
 </instances>
