File: pic_k42.sch (EAGLE design)
At the start: 88 parts, among them IC1 PIC18F57K42-E_PT, IC2 REF3440IDBVR, IC3 MAX232, IC4 ILAMP, J1 MLE-105-01-G-DV, K1 G6K-2P, P10_V 10 volts, Q1 ASF1, U1 LM78L05ACMX/NOPB, X1 RX-2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

Commit message: up
Parts:
- R12: value 220 -> 56
- R13, R9: value 3K -> 3.83K
Changed lines of the file:
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@@
 <part name="TP2" library="testpad" library_urn="urn:adsk.eagle:library:385" deviceset="TP" device="B1,27" package3d_urn="urn:adsk.eagle:package:27944/2"/>
 <part name="VDD10" library="supply1" library_urn="urn:adsk.eagle:library:371" deviceset="VDD" device=""/>
-<part name="R12" library="rcl" library_urn="urn:adsk.eagle:library:334" deviceset="R-US_" device="R1206" package3d_urn="urn:adsk.eagle:package:23540/2" value="220"/>
+<part name="R12" library="rcl" library_urn="urn:adsk.eagle:library:334" deviceset="R-US_" device="R1206" package3d_urn="urn:adsk.eagle:package:23540/2" value="56"/>
 <part name="VSS16" library="supply1" library_urn="urn:adsk.eagle:library:371" deviceset="VSS" device=""/>
 <part name="F1" library="polyfuse-smd_10" deviceset="?" device="1206L" technology="050"/>
@@
 <part name="LED2" library="led" library_urn="urn:adsk.eagle:library:259" deviceset="LED" device="CHIPLED_1206" package3d_urn="urn:adsk.eagle:package:15823/2" value="-15"/>
 <part name="LED4" library="led" library_urn="urn:adsk.eagle:library:259" deviceset="LED" device="CHIPLED_1206" package3d_urn="urn:adsk.eagle:package:15823/2" value="+15"/>
-<part name="R9" library="rcl" library_urn="urn:adsk.eagle:library:334" deviceset="R-US_" device="R1206" package3d_urn="urn:adsk.eagle:package:23540/2" value="3K"/>
-<part name="R13" library="rcl" library_urn="urn:adsk.eagle:library:334" deviceset="R-US_" device="R1206" package3d_urn="urn:adsk.eagle:package:23540/2" value="3K"/>
+<part name="R9" library="rcl" library_urn="urn:adsk.eagle:library:334" deviceset="R-US_" device="R1206" package3d_urn="urn:adsk.eagle:package:23540/2" value="3.83K"/>
+<part name="R13" library="rcl" library_urn="urn:adsk.eagle:library:334" deviceset="R-US_" device="R1206" package3d_urn="urn:adsk.eagle:package:23540/2" value="3.83K"/>
 <part name="VSS51" library="supply1" library_urn="urn:adsk.eagle:library:371" deviceset="VSS" device=""/>
 <part name="VSS52" library="supply1" library_urn="urn:adsk.eagle:library:371" deviceset="VSS" device=""/>
@@
 </instance>
 <instance part="R2" gate="G$1" x="53.34" y="-10.16" smashed="yes" rot="R180">
-<attribute name="NAME" x="57.15" y="-11.6586" size="1.778" layer="95" rot="R180"/>
+<attribute name="NAME" x="52.07" y="-11.6586" size="1.778" layer="95" rot="R180"/>
 <attribute name="VALUE" x="57.15" y="-6.858" size="1.778" layer="96" rot="R180"/>
 </instance>
@@
 </instance>
 <instance part="R12" gate="G$1" x="58.42" y="-5.08" smashed="yes" rot="R90">
-<attribute name="NAME" x="56.9214" y="-8.89" size="1.778" layer="95" rot="R90"/>
-<attribute name="VALUE" x="61.722" y="-8.89" size="1.778" layer="96" rot="R90"/>
+<attribute name="NAME" x="56.9214" y="-6.35" size="1.778" layer="95" rot="R90"/>
+<attribute name="VALUE" x="61.722" y="-6.35" size="1.778" layer="96" rot="R90"/>
 </instance>
 <instance part="VSS16" gate="G$1" x="-7.62" y="-50.8" smashed="yes">

Commit message: up
Connections:
- net N$38 renamed RA1
- net N$39 renamed RA0
- net N$54 renamed ANRB2
- net N$66 renamed ANRB3
Changed lines of the file:
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@@
 </segment>
 </net>
-<net name="N$38" class="0">
+<net name="RA1" class="0">
 <segment>
 <pinref part="IC1" gate="G$1" pin="RA1"/>
@@
 <junction x="83.82" y="35.56"/>
 <junction x="63.5" y="17.78"/>
-<label x="86.36" y="7.62" size="1.778" layer="95"/>
+<label x="83.82" y="5.08" size="1.778" layer="95"/>
 </segment>
 <segment>
@@
 </segment>
 </net>
-<net name="N$39" class="0">
+<net name="RA0" class="0">
 <segment>
 <pinref part="IC1" gate="G$1" pin="RA0"/>
@@
 </segment>
 </net>
-<net name="N$54" class="0">
+<net name="ANRB2" class="0">
 <segment>
 <pinref part="IC1" gate="G$1" pin="RB2"/>
@@
 </segment>
 </net>
-<net name="N$66" class="0">
+<net name="ANRB3" class="0">
 <segment>
 <pinref part="X7" gate="-3" pin="S"/>
@@
 <wire x1="-170.18" y1="-5.08" x2="-177.8" y2="-5.08" width="0.1524" layer="91"/>
 <junction x="-170.18" y="-5.08"/>
-<label x="-177.8" y="-5.08" size="1.778" layer="95"/>
-</segment>
-<segment>
+<label x="-157.48" y="-5.08" size="1.778" layer="95"/>
+</segment>
+<segment>
